Commit message: Trying to fix URDF model. Wheel joints were set to fixed, adding steering joints, etc.

File: ros2_ws/src/simulations/jetrover_description/urdf/car_acker.urdf.xacro (robot description, xacro)
@@ -102,5 +102,5 @@
     <inertial>
       <origin
-        xyz="-0.213334280297957 -0.203369638948946 -0.000334615151787748"
+        xyz="0.213334280297957 0.203369638948946 -0.000334615151787748"
         rpy="0 0 0" />
       <mass
@@ -135,15 +135,48 @@
   </link>
   <joint
+    name="wheel_left_front_steering_joint"
+    type="revolute">
+    <origin
+      xyz="0.106579884267788 0.0916974467397005 -0.0654867643253843"
+      rpy="0 0 0" />
+    <parent
+      link="base_link" />
+    <child
+      link="wheel_left_front_base" />
+    <axis
+      xyz="0 0 1" />
+    <limit effort="100" velocity="1" lower="-0.5" upper="0.5"/>
+  </joint>
+  <link name="wheel_left_front_base">
+    <visual>
+      <origin
+        xyz="0 0 0"
+        rpy="0 0 0" />
+      <geometry>
+        <sphere radius="0.001"/>
+      </geometry>
+      <material name="black"/>
+    </visual>
+    <collision>
+      <origin
+        xyz="0 0 0"
+        rpy="0 0 0" />
+      <geometry>
+        <sphere radius="0.001"/>
+      </geometry>
+    </collision>
+  </link>
+  <joint
     name="wheel_left_front_joint"
     type="continuous">
     <origin
-      xyz="-0.106579884267788 -0.0916974467397005 -0.0654867643253843"
+      xyz="0 0 0"
       rpy="0 0 3.14159265358979" />
     <parent
-      link="base_link" />
+      link="wheel_left_front_base" />
     <child
       link="wheel_left_front_link" />
     <axis
-      xyz="0 0 0" />
+      xyz="0 -1 0" />
   </joint>
   <link
@@ -151,5 +184,5 @@
     <inertial>
       <origin
-        xyz="0.213327728411634 -0.202539554308172 0.000327384188806199"
+        xyz="-0.213327728411634 0.202539554308172 0.000327384188806199"
         rpy="0 0 0" />
       <mass
@@ -187,5 +220,5 @@
     type="continuous">
     <origin
-      xyz="0.106753653016542 -0.0920004072996187 -0.0658214520621466"
+      xyz="-0.106753653016542 0.0920004072996187 -0.0658214520621466"
       rpy="0 0 3.14158803228829" />
     <parent
@@ -194,5 +227,5 @@
       link="wheel_left_back_link" />
     <axis
-      xyz="0 0 0" />
+      xyz="0 -1 0" />
   </joint>
   <link
@@ -200,5 +233,5 @@
     <inertial>
       <origin
-        xyz="-0.213332807255404 0.203675464611681 -0.000332210127461456"
+        xyz="0.213332807255404 -0.203675464611681 -0.000332210127461456"
         rpy="0 0 0" />
       <mass
@@ -233,15 +266,49 @@
   </link>
   <joint
+    name="wheel_right_front_steering_joint"
+    type="revolute">
+    <origin
+      xyz="0.10658 -0.091851 -0.065487"
+      rpy="0 0 0" />
+    <parent
+      link="base_link" />
+    <child
+      link="wheel_right_front_base" />
+    <axis
+      xyz="0 0 1" />
+    <limit effort="100" velocity="1" lower="-0.5" upper="0.5"/>
+  </joint>
+  <link name="wheel_right_front_base">
+    <visual>
+      <origin
+        xyz="0 0 0"
+        rpy="0 0 0" />
+      <geometry>
+        <sphere radius="0.001"/>
+      </geometry>
+      <material name="black"/>
+    </visual>
+    <collision>
+      <origin
+        xyz="0 0 0"
+        rpy="0 0 0" />
+      <geometry>
+        <sphere radius="0.001"/>
+      </geometry>
+    </collision>
+  </link>
+  <joint
     name="wheel_right_front_joint"
     type="continuous">
     <origin
-      xyz="-0.10658 0.091851 -0.065487"
+      xyz="0 0 0"
       rpy="0 0 3.1416" />
     <parent
-      link="base_link" />
+      link="wheel_right_front_base" />
     <child
       link="wheel_right_front_link" />
     <axis
-      xyz="0 0 0" />
+      xyz="0 -1 0" />
+    <limit effort="100" velocity="1"/>
   </joint>
   <link
@@ -249,5 +316,5 @@
     <inertial>
       <origin
-        xyz="0.21333 0.20224 0.00032742"
+        xyz="-0.21333 -0.20224 0.00032742"
         rpy="0 0 0" />
       <mass
@@ -285,5 +352,5 @@
     type="continuous">
     <origin
-      xyz="0.10675 0.091848 -0.065821"
+      xyz="-0.10675 -0.091848 -0.065821"
       rpy="0 0 3.1416" />
     <parent
@@ -292,5 +359,5 @@
       link="wheel_right_back_link" />
     <axis
-      xyz="0 0 0" />
+      xyz="0 -1 0" />
   </joint>
 </robot>

File: ros2_ws/src/simulations/jetrover_description/urdf/gazebo_control.xacro (robot description, xacro)
@@ -3,5 +3,5 @@
     <gazebo>
         <plugin name='gz::sim::systems::AckermannSteering'
-            filename='gz-sim-ackermann-steering-system'>
+        filename='ignition-gazebo-ackermann-steering-system'>
             <left_joint>wheel_left_rear_joint</left_joint>
             <right_joint>wheel_right_rear_joint</right_joint>
@@ -11,9 +11,9 @@
                 </right_steering_joint>
             <!-- TODO: Update Geometry -->
-            <wheel_separation>1.25</wheel_separation>
-            <wheel_radius>0.3</wheel_radius>
-            <kingpin_width>1.0</kingpin_width>
+            <wheel_separation>0.222</wheel_separation>
+            <wheel_radius>0.101</wheel_radius>
+            <kingpin_width>0.2</kingpin_width>
             <steering_limit>0.5</steering_limit>
-            <wheel_base>1.0</wheel_base> <!-- Front-back wheel base -->
+            <wheel_base>0.213</wheel_base> <!-- Front-back wheel base -->
             <min_velocity>-1</min_velocity>
             <max_velocity>1</max_velocity>
@@ -26,6 +26,10 @@
         <plugin name="gz::sim::systems::JointStatePublisher" filename="gz-sim-joint-state-publisher-system">
             <topic>joint_states</topic>
-            <joint_name>left_wheel_joint</joint_name>
-            <joint_name>right_wheel_joint</joint_name>
+            <joint_name>wheel_left_rear_joint</joint_name>
+            <joint_name>wheel_right_rear_joint</joint_name>
+            <joint_name>wheel_left_front_joint</joint_name>
+            <joint_name>wheel_right_front_joint</joint_name>
+            <joint_name>wheel_left_front_steering_joint</joint_name>
+            <joint_name>wheel_right_front_steering_joint</joint_name>
         </plugin>
     </gazebo>
